Commit message: scene for [first demo]

File: urdf/archiv/ur5.urdf (robot description, URDF)
Before this commit: robot ur5, 13 links, 12 joints
Joints:
- joint rg2_eef_joint: origin xyz=0.195 0.0 0.0 rpy=0 1.5707963268 0 -> xyz=0.195 0.0 0.0 rpy=0 0 0
- joint world_joint: origin xyz=0.0 0.0 0.1 rpy=0.0 0.0 0.0 -> xyz=0.0 0.0 0.0 rpy=0.0 0.0 0.0
